File: gonioreflectometer/hw/gonioreflectometer.kicad_sch (KiCad schematic)
At the start: 44 parts, among them Q1 SS8050 200-350, Q10 AO3401A, Q2 SS8050 200-350, Q3 SS8050 200-350, Q4 AO3401A, Q5 AO3400A, Q6 AO3401A, Q7 AO3401A, Q8 AO3401A, Q9 SS8050 200-350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

Commit message: v1.1 compacter (contains drc errors)
Parts:
- removed TP1: 3.3v, TestPoint:TestPoint_Plated_Hole_D2.0mm, symbol Connector:TestPoint
- removed TP2: 5v, TestPoint:TestPoint_Plated_Hole_D2.0mm, symbol Connector:TestPoint
- removed TP3: GND, TestPoint:TestPoint_Plated_Hole_D2.0mm, symbol Connector:TestPoint
- removed TP4: SWD, TestPoint:TestPoint_Plated_Hole_D2.0mm, symbol Connector:TestPoint
- removed TP5: SWCLK, TestPoint:TestPoint_Plated_Hole_D2.0mm, symbol Connector:TestPoint
- removed TP6: Reset, TestPoint:TestPoint_Plated_Hole_D2.0mm, symbol Connector:TestPoint
- removed TP7: USART, TestPoint:TestPoint_Plated_Hole_D2.0mm, symbol Connector:TestPoint
- added J1, J2: Conn_01x07_Pin, Connector_PinHeader_2.54mm:PinHeader_1x07_P2.54mm_Vertical, symbol Connector:Conn_01x07_Pin
Connections:
- net 1_Wire_USART: now also J1.4 (Pin_4), J2.4 (Pin_4)
- net 3.3v: now also J1.2 (Pin_2), J2.2 (Pin_2)
- net 5v: now also J1.1 (Pin_1), J2.1 (Pin_1)
- net Blue_LED_Switch: now also U1.16 (PA8); no longer U1.9 (PA3)
- net GND: now also J1.3 (Pin_3)
- net Green_LED_Switch: now also U1.2 (PA12); no longer U1.11 (PA5)
- net NEXT_GND: now also J2.3 (Pin_3)
- net Red_LED_Switch: now also U1.1 (PB1); no longer U1.10 (PA4)
- net Reset: now also J1.7 (Pin_7), J2.7 (Pin_7)
- net SWCLK: now also J1.6 (Pin_6), J2.6 (Pin_6)
- net SWD: now also J1.5 (Pin_5), J2.5 (Pin_5)
Other:
- note added: "In"
- note added: "Out"
